File: Wiring Diagrams/Capstone V3/power_breakout.sch (EAGLE design)
At the start: 24 parts, among them J1 RASPBERRYPI-40-PIN-GPIO_PTH_N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, U1 2N7000RLRAG

Commit message: Modified power supply board to remove extra holes
Parts:
- removed U$1: POWERBOOST500C, jos-ph:POWERBOOST500C
Connections:
- net GND: no longer U$1.GND1, U$1.GND3
- net N$30: no longer U$1.5V
- net N$4: no longer U$1.LB
- net N$5: no longer U$1.GND2
- net N$6: no longer U$1.EN
- net N$7: no longer U$1.USBIN
- net V_BATT: no longer U$1.BAT
Changed lines of the file:
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@@
 <attribute name="DESIGNER" value="Lesley Wheat"/>
 </part>
-<part name="U$1" library="jos-ph" deviceset="POWERBOOST500C" device=""/>
 <part name="SUPPLY4" library="SparkFun-PowerSymbols" deviceset="5V" device=""/>
 <part name="GND5" library="SparkFun-PowerSymbols" deviceset="GND" device=""/>
@@
 <attribute name="DESIGNER" x="170.434" y="11.176" size="2.7432" layer="94" font="vector"/>
 </instance>
-<instance part="U$1" gate="G$1" x="196.85" y="167.64" smashed="yes" rot="R90"/>
 <instance part="SUPPLY4" gate="G$1" x="144.78" y="157.48" smashed="yes">
 <attribute name="VALUE" x="144.78" y="160.274" size="1.778" layer="96" align="bottom-center"/>
@@
 </segment>
 <segment>
-<pinref part="U$1" gate="G$1" pin="GND3"/>
-<wire x1="189.23" y1="152.4" x2="189.23" y2="115.57" width="0.1524" layer="91"/>
+<wire x1="189.23" y1="179.07" x2="189.23" y2="115.57" width="0.1524" layer="91"/>
 <wire x1="201.93" y1="115.57" x2="189.23" y2="115.57" width="0.1524" layer="91"/>
-<pinref part="U$1" gate="G$1" pin="GND1"/>
-<wire x1="201.93" y1="152.4" x2="201.93" y2="115.57" width="0.1524" layer="91"/>
+<wire x1="201.93" y1="179.07" x2="201.93" y2="115.57" width="0.1524" layer="91"/>
 <pinref part="R3" gate="G$1" pin="1"/>
 <wire x1="163.83" y1="107.95" x2="182.88" y2="107.95" width="0.1524" layer="91"/>
@@
 <junction x="182.88" y="107.95"/>
 <pinref part="JP2" gate="A" pin="2"/>
-<wire x1="189.23" y1="152.4" x2="189.23" y2="179.07" width="0.1524" layer="91"/>
-<junction x="189.23" y="152.4"/>
 <pinref part="JP2" gate="A" pin="7"/>
-<wire x1="201.93" y1="152.4" x2="201.93" y2="179.07" width="0.1524" layer="91"/>
-<junction x="201.93" y="152.4"/>
 </segment>
 </net>
@@
 <pinref part="S1" gate="1" pin="O"/>
 <wire x1="186.69" y1="139.7" x2="180.34" y2="139.7" width="0.1524" layer="91"/>
-<pinref part="U$1" gate="G$1" pin="5V"/>
-<wire x1="186.69" y1="139.7" x2="186.69" y2="152.4" width="0.1524" layer="91"/>
 <pinref part="JP2" gate="A" pin="1"/>
-<wire x1="186.69" y1="152.4" x2="186.69" y2="179.07" width="0.1524" layer="91"/>
-<junction x="186.69" y="152.4"/>
+<wire x1="186.69" y1="139.7" x2="186.69" y2="179.07" width="0.1524" layer="91"/>
 </segment>
 </net>
@@
 <segment>
 <pinref part="SUPPLY8" gate="G$1" pin="V_BATT"/>
-<pinref part="U$1" gate="G$1" pin="BAT"/>
-<wire x1="199.39" y1="152.4" x2="199.39" y2="151.13" width="0.1524" layer="91"/>
 <wire x1="199.39" y1="151.13" x2="199.39" y2="139.7" width="0.1524" layer="91"/>
 <wire x1="199.39" y1="139.7" x2="217.17" y2="139.7" width="0.1524" layer="91"/>
@@
 <label x="111.76" y="153.67" size="1.778" layer="95" rot="R90"/>
 <pinref part="JP2" gate="A" pin="6"/>
-<wire x1="199.39" y1="152.4" x2="199.39" y2="179.07" width="0.1524" layer="91"/>
-<junction x="199.39" y="152.4"/>
+<wire x1="199.39" y1="151.13" x2="199.39" y2="179.07" width="0.1524" layer="91"/>
 <pinref part="JP1" gate="A" pin="3"/>
 <wire x1="104.14" y1="177.8" x2="104.14" y2="172.72" width="0.1524" layer="91"/>
@@
 <net name="N$4" class="0">
 <segment>
-<pinref part="U$1" gate="G$1" pin="LB"/>
 <pinref part="JP2" gate="A" pin="3"/>
 <wire x1="191.77" y1="152.4" x2="191.77" y2="179.07" width="0.1524" layer="91"/>
@@
 <net name="N$5" class="0">
 <segment>
-<pinref part="U$1" gate="G$1" pin="GND2"/>
 <pinref part="JP2" gate="A" pin="4"/>
 <wire x1="194.31" y1="152.4" x2="194.31" y2="179.07" width="0.1524" layer="91"/>
@@
 <net name="N$6" class="0">
 <segment>
-<pinref part="U$1" gate="G$1" pin="EN"/>
 <pinref part="JP2" gate="A" pin="5"/>
 <wire x1="196.85" y1="152.4" x2="196.85" y2="179.07" width="0.1524" layer="91"/>
@@
 <net name="N$7" class="0">
 <segment>
-<pinref part="U$1" gate="G$1" pin="USBIN"/>
 <pinref part="JP2" gate="A" pin="8"/>
 <wire x1="204.47" y1="152.4" x2="204.47" y2="179.07" width="0.1524" layer="91"/>
