File: Wiring Diagrams/Capstone V3/Transponder.brd (EAGLE design)
At the start: 39.7 x 72.4 mm, 22 parts, among them IC1 MCP1700-5002E/TO-ND, IC2 MCP1700-3302E/TO-ND, J1 ARD_H1, J2 ARD_H2, U2 2N7000RLRAG

Commit message: Changed transponder power source from one CR2032 to two CR2032
Parts:
- BT1: value 3.0 -> 6.0
- R4: value 10 -> 47
Changed lines of the file:
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@@
 <?xml version="1.0" encoding="utf-8"?>
 <!DOCTYPE eagle SYSTEM "eagle.dtd">
-<eagle version="9.5.1">
+<eagle version="9.5.2">
 <drawing>
 <settings>
@@
 </autorouter>
 <elements>
-<element name="BT1" library="SparkFun-Batteries" package="BATTCON_20MM_4LEGS" value="3.0" x="31.75" y="13.97" smashed="yes" rot="MR270">
+<element name="BT1" library="SparkFun-Batteries" package="BATTCON_20MM_4LEGS" value="6.0" x="31.75" y="13.97" smashed="yes" rot="MR270">
 <attribute name="NAME" x="24.257" y="13.97" size="0.6096" layer="26" font="vector" ratio="20" rot="MR270" align="bottom-center"/>
 <attribute name="PROD_ID" value="BATT-10373" x="41.91" y="-38.1" size="1.778" layer="28" rot="MR270" display="off"/>
@@
 <attribute name="VALUE" x="36.8808" y="58.674" size="1.27" layer="27" ratio="10" rot="R90"/>
 </element>
-<element name="R4" library="resistor" package="0207/12" value="10" x="33.02" y="63.5" smashed="yes" rot="R270">
+<element name="R4" library="resistor" package="0207/12" value="47" x="33.02" y="63.5" smashed="yes" rot="R270">
 <attribute name="NAME" x="34.417" y="66.675" size="1.27" layer="25" ratio="10" rot="R270"/>
 <attribute name="VALUE" x="32.3342" y="65.786" size="1.27" layer="27" ratio="10" rot="R270"/>
