File: Wiring Diagrams/Capstone V3/Transponder.sch (EAGLE design)
At the start: 22 parts, among them IC1 MCP1700-5002E/TO-ND, IC2 MCP1700-3302E/TO-ND, J1 ARD_H1, J2 ARD_H2, U2 2N7000RLRAG

Commit message: Changed transponder power source from one CR2032 to two CR2032
Parts:
- BT1: value 3.0 -> 6.0
- R4: value 10 -> 47
Changed lines of the file:
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@@
 <?xml version="1.0" encoding="utf-8"?>
 <!DOCTYPE eagle SYSTEM "eagle.dtd">
-<eagle version="9.5.1">
+<eagle version="9.5.2">
 <drawing>
 <settings>
@@
 </classes>
 <parts>
-<part name="BT1" library="SparkFun-Batteries" deviceset="BATTERY" device="-20MM_SMD_4LEGS" value="3.0"/>
+<part name="BT1" library="SparkFun-Batteries" deviceset="BATTERY" device="-20MM_SMD_4LEGS" value="6.0"/>
 <part name="U$1" library="adafruit" deviceset="ARDUINOMICRO" device=""/>
 <part name="U$2" library="adafruit" deviceset="XBEE" device=""/>
@@
 <part name="LED1" library="led" deviceset="LED" device="5MM" value="POWERLED"/>
 <part name="R3" library="resistor" deviceset="R-US_" device="0207/12" value="47"/>
-<part name="R4" library="resistor" deviceset="R-US_" device="0207/12" value="10"/>
+<part name="R4" library="resistor" deviceset="R-US_" device="0207/12" value="47"/>
 <part name="GND3" library="SparkFun-PowerSymbols" deviceset="GND" device=""/>
 <part name="J1" library="SparkFun-Connectors" deviceset="CONN_17" device="NOSILK" value="ARD_H1"/>
